Commit message: finish all tasks

File: xacro/rb1_ros2_base.urdf.xacro (robot description, xacro)
@@ -125,5 +125,5 @@
     <gazebo>
 		<plugin name="elevator_controller" filename="libgazebo_ros_force_system.so">
-			 <link name="$(arg prefix)elevator_platform" />
+			 <link name="robot_elevator_base_link" />
             <force>
 			    <x>0</x>
@@ -131,4 +131,5 @@
                 <z>10</z> <!-- Adjust the force as per your requirement -->
             </force>
+             <update_rate>100</update_rate>
 		</plugin>
 	</gazebo>
